File: AART11-2023-12-13_115145/s001.kicad_sch (KiCad schematic)
At the start: 39 parts, among them J10 Conn_01x01_Pin, J11 Conn_01x01_Pin, J2 Conn_01x01_Pin, J3 Conn_01x01_Pin, J8 Conn_01x01_Pin, J9 Conn_01x01_Pin, U3 FD6288Q

Commit message: Updated v8 fix footprints
Parts:
- Q? (x6): footprint Package_SON:VSON-8_3.3x3.3mm_P0.65mm_NexFET -> Package_TO_SOT_SMD:TDSON-8-1
- U3: symbol Portia:FD6288Q -> LibProj:FD6288Q
- gave numbers to parts that had none: 26
