File: AART11-2023-12-13_115145/s002.kicad_sch (KiCad schematic)
At the start: 13 parts, among them J1 Conn_01x01_Pin, J4 Conn_01x04, J5 Conn_01x01, J6 Conn_01x01, J7 Conn_01x01, U4 AT32F421G8U7

Commit message: Updated v8 fix footprints
Parts:
- U4: footprint Package_DFN_QFN:QFN-28-1EP_4x4mm_P0.4mm_EP2.6x2.6mm -> Package_DFN_QFN:QFN-28-1EP_4x4mm_P0.4mm_EP2.3x2.3mm_ThermalVias
- gave numbers to parts that had none: 7
