File: AART11-2023-12-13_115145/AART11.kicad_pcb (KiCad board)
At the start: 4 copper layers, 16.2 x 23.2 mm, 82 parts, among them J1 Conn_01x01_Pin, J10 Conn_01x01_Pin, J11 Conn_01x01_Pin, J2 Conn_01x01_Pin, J3 Conn_01x01_Pin, J4 Conn_01x04, J5 Conn_01x01, J6 Conn_01x01, J7 Conn_01x01, J8 Conn_01x01_Pin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

Commit message: Updated v8 fix footprints
Parts:
- Q10, Q4, Q5, Q6, Q7, Q8, Q9: footprint Package_SON:VSON-8_3.3x3.3mm_P0.65mm_NexFET -> Package_TO_SOT_SMD:TDSON-8-1
- U4: footprint Package_DFN_QFN:QFN-28-1EP_4x4mm_P0.4mm_EP2.6x2.6mm -> Package_DFN_QFN:QFN-28-1EP_4x4mm_P0.4mm_EP2.3x2.3mm_ThermalVias
- renumbered + to TP5
Connections:
- J4 pad : GND -> (no net)
- U3 pad 8: unconnected-(U3-NC-Pad8) -> (no net)

Commit message: Added inductor fp
Parts:
- L1: footprint Inductor_SMD:L_Taiyo-Yuden_MD-2020 -> Added_footprints:L_Sunltech_SLW201610P
Changed lines of the file:
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@@
 		)
 	)
-	(footprint "Inductor_SMD:L_Taiyo-Yuden_MD-2020"
+	(footprint "Added_footprints:L_Sunltech_SLW201610P"
 		(layer "B.Cu")
 		(at 166.275 125.025 180)
@@
 		(tags "inductor taiyo-yuden md smd")
 		(property "Reference" "L1"
-			(at 0 2 0)
+			(at 0 2 180)
 			(layer "B.SilkS")
 			(hide yes)
@@
 		)
 		(property "Value" "10uH"
-			(at 0 -2.5 0)
+			(at 0 -2.5 180)
 			(layer "B.Fab")
 			(effects
@@
 			)
 		)
-		(property "Footprint" "Inductor_SMD:L_Taiyo-Yuden_MD-2020"
+		(property "Footprint" "Added_footprints:L_Sunltech_SLW201610P"
 			(at 0 0 180)
 			(unlocked yes)
@@
 		)
 		(property "JLCPCB Part #" "C207862"
-			(at 0 0 0)
+			(at 0 0 180)
 			(layer "B.Fab")
 			(hide yes)
@@
 		)
 		(property "Rating" "750mA - ±20%"
-			(at 0 0 0)
+			(at 0 0 180)
 			(layer "B.Fab")
 			(hide yes)
@@
 		(attr smd)
 		(fp_line
-			(start 1.3 1.3)
-			(end -1.3 1.3)
+			(start 1.36 1.15)
+			(end -1.36 1.15)
 			(stroke
 				(width 0.05)
@@
 		)
 		(fp_line
-			(start 1.3 -1.3)
-			(end 1.3 1.3)
+			(start 1.36 -1.15)
+			(end 1.36 1.15)
 			(stroke
 				(width 0.05)
@@
 		)
 		(fp_line
-			(start -1.3 1.3)
-			(end -1.3 -1.3)
+			(start -1.36 1.15)
+			(end -1.36 -1.15)
 			(stroke
 				(width 0.05)
@@
 		)
 		(fp_line
-			(start -1.3 -1.3)
-			(end 1.3 -1.3)
+			(start -1.36 -1.15)
+			(end 1.36 -1.15)
 			(stroke
 				(width 0.05)
@@
 		)
 		(fp_line
-			(start 1 1)
-			(end -1 1)
+			(start 1 0.8)
+			(end -1 0.8)
 			(stroke
 				(width 0.1)
@@
 		)
 		(fp_line
-			(start 1 -1)
-			(end 1 1)
+			(start 1 -0.8)
+			(end 1 0.8)
 			(stroke
 				(width 0.1)
@@
 		)
 		(fp_line
-			(start -1 1)
-			(end -1 -1)
+			(start -1 0.8)
+			(end -1 -0.8)
 			(stroke
 				(width 0.1)
@@
 		)
 		(fp_line
-			(start -1 -1)
-			(end 1 -1)
+			(start -1 -0.8)
+			(end 1 -0.8)
 			(stroke
 				(width 0.1)
@@
 		)
 		(fp_text user "${REFERENCE}"
-			(at 0 0 0)
+			(at 0 0 180)
 			(layer "B.Fab")
 			(effects
@@
 		)
 		(pad "1" smd rect
-			(at -0.675 0 180)
-			(size 0.65 2)
+			(at -0.66 0 180)
+			(size 0.89 1.42)
 			(layers "B.Cu" "B.Paste" "B.Mask")
 			(net 5 "VDC")
@@
 		)
 		(pad "2" smd rect
-			(at 0.675 0 180)
-			(size 0.65 2)
+			(at 0.66 0 180)
+			(size 0.89 1.42)
 			(layers "B.Cu" "B.Paste" "B.Mask")
 			(net 16 "Net-(D4-A)")
