File: AART11-2023-12-13_115145/AART11.kicad_sch (KiCad schematic)
At the start: 30 parts, among them Q1 FMMT718, Q2 EMZ1T2R, Q3 MMBFJ309, U1 AP3015KTR-G1, U2 AP2210K-3.3TRG1

Commit message: Updated v8 fix footprints
Parts:
- Q?: footprint Package_SON:VSON-8_3.3x3.3mm_P0.65mm_NexFET -> Package_TO_SOT_SMD:TDSON-8-1

Commit message: Added inductor fp
Parts:
- L1: footprint Inductor_SMD:L_Taiyo-Yuden_MD-2020 -> Added_footprints:L_Sunltech_SLW201610P
Changed lines of the file:
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@@
 			)
 		)
-		(property "Footprint" "Inductor_SMD:L_Taiyo-Yuden_MD-2020"
+		(property "Footprint" "Added_footprints:L_Sunltech_SLW201610P"
 			(at 69.85 114.3 0)
 			(effects
