File: MidA/MidA.kicad_pcb (KiCad board)
At the start: 4 copper layers, 16.2 x 23.2 mm, 82 parts, among them J1 Conn_01x01_Pin, J10 Conn_01x01_Pin, J11 Conn_01x01_Pin, J2 Conn_01x01_Pin, J3 Conn_01x01_Pin, J4 Conn_01x04, J5 Conn_01x01, J6 Conn_01x01, J7 Conn_01x01, J8 Conn_01x01_Pin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

Commit message: Added pkg
Parts:
- added G***: LOGO, MidA:logo, B.Cu at (170.5, 117.0)
Other:
- board text removed: "AART"
- board text removed: "Remora1"
