File: AART11/AART11.kicad_sch (KiCad schematic)
At the start: 30 parts, among them Q1 FMMT718, Q2 EMZ1T2R, Q3 MMBFJ309, U1 AP3015KTR-G1, U2 AP2210K-3.3TRG1

Commit message: Better fets
Parts:
- Q?: value AON7418 -> JMSL0302AU

Commit message: Wrong part number
Parts:
- Q?: JLCPCB Part # C74384 -> C2890409
Changed lines of the file:
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@@
 			)
 		)
-		(property "JLCPCB Part #" "C74384"
+		(property "JLCPCB Part #" "C2890409"
 			(at 63.5 86.36 0)
 			(effects

Commit message: KiCad 9 update
Parts:
- gave numbers to parts that had none: 1
Changed lines of the file:
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@@
 (kicad_sch
-	(version 20231120)
+	(version 20250114)
 	(generator "eeschema")
-	(generator_version "8.0")
+	(generator_version "9.0")
 	(paper "A4")
 	(title_block
@@
 		(company "ECOM")
 	)
+	(text "3V366 ~ 3V234"
+		(exclude_from_sim no)
+		(at 90.17 167.64 0)
+		(effects
+			(font
+				(size 1.27 1.27)
+			)
+			(justify left bottom)
+		)
+	)
+	(text "9V~12V"
+		(exclude_from_sim no)
+		(at 144.78 25.4 0)
+		(effects
+			(font
+				(size 1.27 1.27)
+			)
+			(justify left bottom)
+		)
+	)
+	(text "1V2~18V"
+		(exclude_from_sim no)
+		(at 35.56 30.48 0)
+		(effects
+			(font
+				(size 1.27 1.27)
+			)
+			(justify right bottom)
+		)
+	)
+	(text "12V4"
+		(exclude_from_sim no)
+		(at 128.27 116.84 0)
+		(effects
+			(font
+				(size 1.27 1.27)
+			)
+			(justify left bottom)
+		)
+	)
 	(junction
 		(at 88.9 127)
@@
 		)
 	)
-	(text "3V366 ~ 3V234"
-		(exclude_from_sim no)
-		(at 90.17 167.64 0)
-		(effects
-			(font
-				(size 1.27 1.27)
-			)
-			(justify left bottom)
-		)
-	)
-	(text "9V~12V"
-		(exclude_from_sim no)
-		(at 144.78 25.4 0)
-		(effects
-			(font
-				(size 1.27 1.27)
-			)
-			(justify left bottom)
-		)
-	)
-	(text "1V2~18V"
-		(exclude_from_sim no)
-		(at 35.56 30.48 0)
-		(effects
-			(font
-				(size 1.27 1.27)
-			)
-			(justify right bottom)
-		)
-	)
-	(text "12V4"
-		(exclude_from_sim no)
-		(at 128.27 116.84 0)
-		(effects
-			(font
-				(size 1.27 1.27)
-			)
-			(justify left bottom)
-		)
-	)
 	(global_label "SVIN"
 		(shape output)
@@
 		(on_board yes)
 		(dnp no)
-		(property "Reference" "Q?"
+		(property "Reference" "Q4"
 			(at 64.77 92.71 90)
 			(effects
@@
 		(at 228.6 63.5)
 		(size 38.1 25.4)
+		(exclude_from_sim no)
+		(in_bom yes)
+		(on_board yes)
+		(dnp no)
 		(fields_autoplaced yes)
 		(stroke
@@
 		(at 228.6 25.4)
 		(size 38.1 25.4)
+		(exclude_from_sim no)
+		(in_bom yes)
+		(on_board yes)
+		(dnp no)
 		(fields_autoplaced yes)
 		(stroke
@@
 		)
 	)
+	(embedded_fonts no)
 )
