File: AART11/s001.kicad_sch (KiCad schematic)
At the start: 39 parts, among them J10 Conn_01x01_Pin, J11 Conn_01x01_Pin, J2 Conn_01x01_Pin, J3 Conn_01x01_Pin, J8 Conn_01x01_Pin, J9 Conn_01x01_Pin, U3 FD6288Q

Commit message: Better fets
Parts:
- Q? (x6): value AP90N03Q -> JMSL0302AU
- gave numbers to parts that had none: 26

Commit message: Wrong part number
Parts:
- Q? (x6): JLCPCB Part # C2828593 -> C2890409
Changed lines of the file:
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@@
 			)
 		)
-		(property "JLCPCB Part #" "C2828593"
+		(property "JLCPCB Part #" "C2890409"
 			(at 149.86 82.55 0)
 			(effects
@@
 			)
 		)
-		(property "JLCPCB Part #" "C2828593"
+		(property "JLCPCB Part #" "C2890409"
 			(at 162.56 95.25 0)
 			(effects
@@
 			)
 		)
-		(property "JLCPCB Part #" "C2828593"
+		(property "JLCPCB Part #" "C2890409"
 			(at 137.16 50.8 0)
 			(effects
@@
 			)
 		)
-		(property "JLCPCB Part #" "C2828593"
+		(property "JLCPCB Part #" "C2890409"
 			(at 149.86 69.85 0)
 			(effects
@@
 			)
 		)
-		(property "JLCPCB Part #" "C2828593"
+		(property "JLCPCB Part #" "C2890409"
 			(at 137.16 63.5 0)
 			(effects
@@
 			)
 		)
-		(property "JLCPCB Part #" "C2828593"
+		(property "JLCPCB Part #" "C2890409"
 			(at 162.56 107.95 0)
 			(effects

Commit message: KiCad 9 update
Parts:
- gave numbers to parts that had none: 6
Changed lines of the file:
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@@
 (kicad_sch
-	(version 20231120)
+	(version 20250114)
 	(generator "eeschema")
-	(generator_version "8.0")
+	(generator_version "9.0")
 	(paper "A4")
 	(title_block
@@
 		(on_board yes)
 		(dnp no)
-		(property "Reference" "Q?"
+		(property "Reference" "Q8"
 			(at 156.21 82.55 0)
 			(effects
@@
 		(on_board yes)
 		(dnp no)
-		(property "Reference" "Q?"
+		(property "Reference" "Q9"
 			(at 168.91 95.25 0)
 			(effects
@@
 		(on_board yes)
 		(dnp no)
-		(property "Reference" "Q?"
+		(property "Reference" "Q5"
 			(at 143.51 50.8 0)
 			(effects
@@
 		(on_board yes)
 		(dnp no)
-		(property "Reference" "Q?"
+		(property "Reference" "Q7"
 			(at 156.21 69.85 0)
 			(effects
@@
 		(on_board yes)
 		(dnp no)
-		(property "Reference" "Q?"
+		(property "Reference" "Q6"
 			(at 143.51 63.5 0)
 			(effects
@@
 		(on_board yes)
 		(dnp no)
-		(property "Reference" "Q?"
+		(property "Reference" "Q10"
 			(at 168.91 107.95 0)
 			(effects
