File: AART11/s002.kicad_sch (KiCad schematic)
At the start: 13 parts, among them J1 Conn_01x01_Pin, J4 Conn_01x04, J5 Conn_01x01, J6 Conn_01x01, J7 Conn_01x01, U4 AT32F421G8U7

Commit message: Better fets
Parts:
- gave numbers to parts that had none: 7
