File: AART11/AART11.kicad_pcb (KiCad board)
At the start: 4 copper layers, 16.2 x 23.2 mm, 82 parts, among them J1 Conn_01x01_Pin, J10 Conn_01x01_Pin, J11 Conn_01x01_Pin, J2 Conn_01x01_Pin, J3 Conn_01x01_Pin, J4 Conn_01x04, J5 Conn_01x01, J6 Conn_01x01, J7 Conn_01x01, J8 Conn_01x01_Pin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

Commit message: Better fets
Parts:
- Q10, Q5, Q6, Q7, Q8, Q9: value AP90N03Q -> JMSL0302AU
- Q4: value AON7418 -> JMSL0302AU
Connections:
- J4 pad : GND -> (no net)
Other:
- board text added: "Remora1.2"
- board text removed: "Remora1"

Commit message: Wrong part number
Parts:
- renumbered + to TP5
Changed lines of the file:
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@@
 			)
 		)
-		(property "JLCPCB Part #" "C2828593"
+		(property "JLCPCB Part #" "C2890409"
 			(at 51.2 266.3 0)
 			(layer "F.Fab")
@@
 			)
 		)
-		(property "JLCPCB Part #" "C2828593"
+		(property "JLCPCB Part #" "C2890409"
 			(at 59.3074 274.4074 0)
 			(layer "F.Fab")
@@
 			)
 		)
-		(property "JLCPCB Part #" "C2828593"
+		(property "JLCPCB Part #" "C2890409"
 			(at 55.263 270.361 0)
 			(layer "F.Fab")
@@
 		(descr "SMD rectangular pad as test Point, square 2.5mm side length")
 		(tags "test point SMD pad rectangle square")
-		(property "Reference" "+"
+		(property "Reference" "TP5"
 			(at -0.02 2.714 0)
 			(layer "B.SilkS")
@@
 			)
 		)
-		(property "JLCPCB Part #" "C2828593"
+		(property "JLCPCB Part #" "C2890409"
 			(at 274.4065 -59.2841 0)
 			(layer "B.Fab")
@@
 			)
 		)
-		(property "JLCPCB Part #" "C2828593"
+		(property "JLCPCB Part #" "C2890409"
 			(at 266.3 -51.2 0)
 			(layer "B.Fab")
@@
 			)
 		)
-		(property "JLCPCB Part #" "C2828593"
+		(property "JLCPCB Part #" "C2890409"
 			(at 270.364 -55.264 0)
 			(layer "B.Fab")
@@
 			)
 		)
-		(property "JLCPCB Part #" "C74384"
+		(property "JLCPCB Part #" "C2890409"
 			(at 0 0 0)
 			(layer "B.Fab")

Commit message: KiCad 9 update
Other:
- board text added: "+"

Commit message: Logo update for e8
Parts:
- added e8-logo: e8-logo, e8-logo:e8, B.Cu at (170.0, 117.0)
Other:
- board text removed: "AART"
- board text removed: "Remora1.2"
